File: hardware/johnson-node/Johnson-node.kicad_sch (KiCad schematic)
At the start: 86 parts, among them IC1 ADC124S051CIMM_NOPB, IC2 ADC124S051CIMM_NOPB, J1 Conn_01x02, J10 Conn_01x03, J11 Conn_01x03, J13 BSEL, J14 RST, J15 SO4B-XASK-1, J16 Conn_01x02, J17 Conn_01x14, J2 Conn_01x03, J3 Conn_01x03, J4 Conn_01x03, J5 Conn_01x03, J6 Conn_01x03, J7 Conn_01x03, J8 Conn_01x03, J9 Conn_01x03, U1 ESP32-S3-WROOM-1U-N4R2, U2 LMR50410Y3FQDBVRQ1, U3 LMR50410Y5FQDBVRQ1, U4 ISO1042BQDWVQ1, U5 MAX3390EEUD_T, U6 MAX3390EEUD_T

Commit message: minor changes
Connections:
- net +12V is gone; now on net BATT: J17.11 (Pin_11), J17.13 (Pin_13)
- net at U1.11 (IO18): now also R18.1
- net at U1.28 (IO35): no longer R18.1
Other:
- moved on the sheet: D11, R18
Changed lines of the file:
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@@
 	)
 	(no_connect
-		(at 347.98 55.88)
-	)
-	(no_connect
 		(at 347.98 93.98)
 	)
@@
 	)
 	(no_connect
+		(at 347.98 66.04)
+	)
+	(no_connect
 		(at 347.98 48.26)
 	)
@@
 	(wire
 		(pts
-			(xy 355.6 66.04) (xy 356.87 66.04)
-		)
-		(stroke
-			(width 0)
-			(type default)
-		)
-	)
-	(wire
-		(pts
 			(xy 360.68 50.8) (xy 370.84 50.8)
 		)
@@
 	(wire
 		(pts
+			(xy 368.3 55.88) (xy 368.3 68.58)
+		)
+		(stroke
+			(width 0)
+			(type default)
+		)
+	)
+	(wire
+		(pts
+			(xy 375.92 68.58) (xy 377.19 68.58)
+		)
+		(stroke
+			(width 0)
+			(type default)
+		)
+	)
+	(wire
+		(pts
 			(xy 82.55 120.65) (xy 90.17 120.65)
 		)
@@
 	(wire
 		(pts
-			(xy 369.57 66.04) (xy 364.49 66.04)
+			(xy 392.43 68.58) (xy 384.81 68.58)
 		)
 		(stroke
@@
 	(wire
 		(pts
+			(xy 347.98 55.88) (xy 368.3 55.88)
+		)
+		(stroke
+			(width 0)
+			(type default)
+		)
+	)
+	(wire
+		(pts
 			(xy 24.13 118.11) (xy 24.13 125.73)
 		)
@@
 	(symbol
 		(lib_id "Device:LED")
-		(at 360.68 66.04 180)
+		(at 381 68.58 180)
 		(unit 1)
 		(body_style 1)
@@
 		(dnp no)
 		(property "Reference" "D11"
-			(at 358.14 67.056 0)
+			(at 378.46 69.596 0)
 			(show_name no)
 			(do_not_autoplace no)
@@
 		)
 		(property "Value" "RED LED"
-			(at 364.744 66.802 0)
+			(at 385.064 69.342 0)
 			(show_name no)
 			(do_not_autoplace no)
@@
 		)
 		(property "Footprint" "LED_SMD:LED_0603_1608Metric"
-			(at 360.68 66.04 0)
+			(at 381 68.58 0)
 			(hide yes)
 			(show_name no)
@@
 		)
 		(property "Datasheet" "https://www.kingbrightusa.com/images/catalog/SPEC/AP2012EC.pdf"
-			(at 360.68 66.04 0)
+			(at 381 68.58 0)
 			(hide yes)
 			(show_name no)
@@
 		)
 		(property "Description" "Light emitting diode"
-			(at 360.68 66.04 0)
+			(at 381 68.58 0)
 			(hide yes)
 			(show_name no)
@@
 		)
 		(property "Sim.Pins" "1=K 2=A"
-			(at 360.68 66.04 0)
+			(at 381 68.58 0)
 			(hide yes)
 			(show_name no)
@@
 		)
 		(property "Part Number" "AP2012EC"
-			(at 360.68 66.04 0)
+			(at 381 68.58 0)
 			(hide yes)
 			(show_name no)
@@
 			)
 		)
-		(property "Value" "+12V"
+		(property "Value" "BATT"
 			(at 242.316 195.58 90)
 			(show_name no)
@@
 	(symbol
 		(lib_id "power:GND")
-		(at 369.57 66.04 0)
+		(at 392.43 68.58 0)
 		(unit 1)
 		(body_style 1)
@@
 		(fields_autoplaced yes)
 		(property "Reference" "#PWR039"
-			(at 369.57 72.39 0)
+			(at 392.43 74.93 0)
 			(hide yes)
 			(show_name no)
@@
 		)
 		(property "Value" "GND"
-			(at 369.57 71.12 0)
+			(at 392.43 73.66 0)
 			(show_name no)
 			(do_not_autoplace no)
@@
 		)
 		(property "Footprint" ""
-			(at 369.57 66.04 0)
+			(at 392.43 68.58 0)
 			(hide yes)
 			(show_name no)
@@
 		)
 		(property "Datasheet" ""
-			(at 369.57 66.04 0)
+			(at 392.43 68.58 0)
 			(hide yes)
 			(show_name no)
@@
 		)
 		(property "Description" "Power symbol creates a global label with name \"GND\" , ground"
-			(at 369.57 66.04 0)
+			(at 392.43 68.58 0)
 			(hide yes)
 			(show_name no)
@@
 			)
 		)
-		(property "Value" "+12V"
+		(property "Value" "BATT"
 			(at 242.316 200.66 90)
 			(show_name no)
@@
 	(symbol
 		(lib_id "Device:R")
-		(at 351.79 66.04 90)
+		(at 372.11 68.58 90)
 		(unit 1)
 		(body_style 1)
@@
 		(dnp no)
 		(property "Reference" "R18"
-			(at 351.79 68.326 90)
+			(at 372.11 70.866 90)
 			(show_name no)
 			(do_not_autoplace no)
@@
 		)
 		(property "Value" "270R"
-			(at 351.79 66.04 90)
+			(at 376.682 71.12 90)
 			(show_name no)
 			(do_not_autoplace no)
@@
 		)
 		(property "Footprint" "Resistor_SMD:R_0603_1608Metric"
-			(at 351.79 67.818 90)
+			(at 372.11 70.358 90)
 			(hide yes)
 			(show_name no)
@@
 		)
 		(property "Datasheet" "https://www.yageogroup.com/content/datasheet/asset/file/PYU-RC_GROUP_51_ROHS_L"
-			(at 351.79 66.04 0)
+			(at 372.11 68.58 0)
 			(hide yes)
 			(show_name no)
@@
 		)
 		(property "Description" "Resistor"
-			(at 351.79 66.04 0)
+			(at 372.11 68.58 0)
 			(hide yes)
 			(show_name no)
@@
 		)
 		(property "Part Number" "RC0805FR-07270RL"
-			(at 351.79 66.04 90)
+			(at 372.11 68.58 90)
 			(hide yes)
 			(show_name no)

Commit message: add onboard reg
Connections:
- net RX: now also J17.9 (Pin_9), U1.5 (IO5); no longer U1.36 (RXD0)
- net TX: now also J17.10 (Pin_10), U1.6 (IO6); no longer U1.37 (TXD0)
- net PPS: now reaches J17.6 (Pin_6)
- net PPS: now also U1.10 (IO17)
- net SCL: now reaches J17.7 (Pin_7)
- net SCL: now also U1.9 (IO16)
- net SDA: now reaches J17.8 (Pin_8)
- net SDA: now also U1.8 (IO15)
- no-connect marks 24 -> 21
Changed lines of the file:
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@@
 	)
 	(no_connect
-		(at 295.91 73.66)
+		(at 347.98 86.36)
 	)
 	(no_connect
-		(at 347.98 86.36)
+		(at 295.91 53.34)
 	)
 	(no_connect
@@
 	)
 	(no_connect
-		(at 347.98 50.8)
-	)
-	(no_connect
 		(at 152.4 119.38)
 	)
@@
 	)
 	(no_connect
-		(at 295.91 71.12)
-	)
-	(no_connect
 		(at 347.98 93.98)
 	)
 	(no_connect
-		(at 347.98 53.34)
+		(at 295.91 50.8)
 	)
 	(no_connect
@@
 	)
 	(no_connect
-		(at 347.98 48.26)
-	)
-	(no_connect
 		(at 347.98 88.9)
 	)
@@
 		)
 	)
-	(global_label "TX"
+	(global_label "SCL"
 		(shape input)
-		(at 295.91 53.34 180)
+		(at 347.98 50.8 0)
 		(fields_autoplaced yes)
 		(effects
@@
 				(size 1.27 1.27)
 			)
-			(justify right)
+			(justify left)
 		)
 		(property "Intersheetrefs" "${INTERSHEET_REFS}"
-			(at 290.7477 53.34 0)
+			(at 354.4728 50.8 0)
 			(hide yes)
 			(show_name no)
@@
 					(size 1.27 1.27)
 				)
-				(justify right)
+				(justify left)
 			)
 		)
@@
 		)
 	)
+	(global_label "TX"
+		(shape input)
+		(at 295.91 73.66 180)
+		(fields_autoplaced yes)
+		(effects
+			(font
+				(size 1.27 1.27)
+			)
+			(justify right)
+		)
+		(property "Intersheetrefs" "${INTERSHEET_REFS}"
+			(at 290.7477 73.66 0)
+			(hide yes)
+			(show_name no)
+			(do_not_autoplace no)
+			(effects
+				(font
+					(size 1.27 1.27)
+				)
+				(justify right)
+			)
+		)
+	)
 	(global_label "5V_CS_C"
 		(shape input)
@@
 		)
 	)
-	(global_label "RX"
+	(global_label "PPS"
 		(shape input)
-		(at 295.91 50.8 180)
+		(at 347.98 53.34 0)
 		(fields_autoplaced yes)
 		(effects
@@
 				(size 1.27 1.27)
 			)
-			(justify right)
+			(justify left)
 		)
 		(property "Intersheetrefs" "${INTERSHEET_REFS}"
-			(at 290.4453 50.8 0)
+			(at 354.7147 53.34 0)
 			(hide yes)
 			(show_name no)
@@
 					(size 1.27 1.27)
 				)
-				(justify right)
+				(justify left)
 			)
 		)
@@
 		)
 	)
+	(global_label "PPS"
+		(shape input)
+		(at 245.11 182.88 180)
+		(fields_autoplaced yes)
+		(effects
+			(font
+				(size 1.27 1.27)
+			)
+			(justify right)
+		)
+		(property "Intersheetrefs" "${INTERSHEET_REFS}"
+			(at 238.3753 182.88 0)
+			(hide yes)
+			(show_name no)
+			(do_not_autoplace no)
+			(effects
+				(font
+					(size 1.27 1.27)
+				)
+				(justify right)
+			)
+		)
+	)
 	(global_label "SGF_P"
 		(shape input)
@@
 		)
 	)
+	(global_label "RX"
+		(shape input)
+		(at 295.91 71.12 180)
+		(fields_autoplaced yes)
+		(effects
+			(font
+				(size 1.27 1.27)
+			)
+			(justify right)
+		)
+		(property "Intersheetrefs" "${INTERSHEET_REFS}"
+			(at 290.4453 71.12 0)
+			(hide yes)
+			(show_name no)
+			(do_not_autoplace no)
+			(effects
+				(font
+					(size 1.27 1.27)
+				)
+				(justify right)
+			)
+		)
+	)
 	(global_label "SGB"
 		(shape input)
@@
 		)
 	)
+	(global_label "RX"
+		(shape input)
+		(at 245.11 190.5 180)
+		(fields_autoplaced yes)
+		(effects
+			(font
+				(size 1.27 1.27)
+			)
+			(justify right)
+		)
+		(property "Intersheetrefs" "${INTERSHEET_REFS}"
+			(at 239.6453 190.5 0)
+			(hide yes)
+			(show_name no)
+			(do_not_autoplace no)
+			(effects
+				(font
+					(size 1.27 1.27)
+				)
+				(justify right)
+			)
+		)
+	)
 	(global_label "SGG"
 		(shape input)
@@
 		)
 	)
+	(global_label "TX"
+		(shape input)
+		(at 245.11 193.04 180)
+		(fields_autoplaced yes)
+		(effects
+			(font
+				(size 1.27 1.27)
+			)
+			(justify right)
+		)
+		(property "Intersheetrefs" "${INTERSHEET_REFS}"
+			(at 239.9477 193.04 0)
+			(hide yes)
+			(show_name no)
+			(do_not_autoplace no)
+			(effects
+				(font
+					(size 1.27 1.27)
+				)
+				(justify right)
+			)
+		)
+	)
 	(global_label "USBD+"
 		(shape input)
@@
 		)
 	)
+	(global_label "SDA"
+		(shape input)
+		(at 245.11 187.96 180)
+		(fields_autoplaced yes)
+		(effects
+			(font
+				(size 1.27 1.27)
+			)
+			(justify right)
+		)
+		(property "Intersheetrefs" "${INTERSHEET_REFS}"
+			(at 238.5567 187.96 0)
+			(hide yes)
+			(show_name no)
+			(do_not_autoplace no)
+			(effects
+				(font
+					(size 1.27 1.27)
+				)
+				(justify right)
+			)
+		)
+	)
 	(global_label "SGG_P"
 		(shape input)
@@
 		)
 	)
+	(global_label "SCL"
+		(shape input)
+		(at 245.11 185.42 180)
+		(fields_autoplaced yes)
+		(effects
+			(font
+				(size 1.27 1.27)
+			)
+			(justify right)
+		)
+		(property "Intersheetrefs" "${INTERSHEET_REFS}"
+			(at 238.6172 185.42 0)
+			(hide yes)
+			(show_name no)
+			(do_not_autoplace no)
+			(effects
+				(font
+					(size 1.27 1.27)
+				)
+				(justify right)
+			)
+		)
+	)
 	(global_label "5V_CS_B"
 		(shape input)
@@
 			)
 		)
+	)
+	(global_label "SDA"
+		(shape input)
+		(at 347.98 48.26 0)
+		(fields_autoplaced yes)
+		(effects
+			(font
+				(size 1.27 1.27)
+			)
+			(justify left)
+		)
+		(property "Intersheetrefs" "${INTERSHEET_REFS}"
+			(at 354.5333 48.26 0)
+			(hide yes)
+			(show_name no)
+			(do_not_autoplace no)
+			(effects
+				(font
+					(size 1.27 1.27)
+				)
+				(justify left)
+			)
+		)

Commit message: 3d models
Parts:
- L1, L2: footprint CustomFootprints:Shielded_Inductor_SMD_7265 -> CustomFootprints:WE-TPC_4828
Changed lines of the file:
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@@
 			)
 		)
-		(property "Footprint" "CustomFootprints:Shielded_Inductor_SMD_7265"
+		(property "Footprint" "CustomFootprints:WE-TPC_4828"
 			(at 64.77 78.74 0)
 			(hide yes)
@@
 			)
 		)
-		(property "Footprint" "CustomFootprints:Shielded_Inductor_SMD_7265"
+		(property "Footprint" "CustomFootprints:WE-TPC_4828"
 			(at 68.58 118.11 0)
 			(hide yes)
