File: hardware/hats/IMU, GPS/IGL.kicad_pcb (KiCad board)
At the start: 2 copper layers, 78 x 58 mm, 9 parts, among them J1 Conn_01x14, J2 GPS, J3 IMU

Commit message: add onboard reg
Parts:
- added C5: 0.22u, Capacitor_SMD:C_0603_1608Metric, F.Cu at (128.5, 63.8)
- added C6: 10u, Capacitor_SMD:C_0603_1608Metric, F.Cu at (128.2, 73.2)
- added U5: BD433, Custom_MSM:Regulator_Linear_SOT-223-4, F.Cu at (128.5, 68.5)
- C1, C3: value C -> 10u
- C2, C4: value C -> 100n
Connections:
- J1 pad 11: +3V3 -> BATT
Routing:
- net BATT: track 0.00 -> 37.5 mm
- net +3V3: track 68.7 -> 74.8 mm
