File: hardware/hats/IMU, GPS/IGL.kicad_sch (KiCad schematic)
At the start: 7 parts, among them J1 Conn_01x14, J2 GPS, J3 IMU

Commit message: add onboard reg
Parts:
- added C5: 0.22u, Capacitor_SMD:C_0603_1608Metric, symbol Device:C
- added C6: 10u, Capacitor_SMD:C_0603_1608Metric, symbol Device:C
- added U5: BD433, Custom_MSM:Regulator_Linear_SOT-223-4, symbol Custom_MSM:Regulator_Linear_5V
- C1, C3: value C -> 10u
- C2, C4: value C -> 100n
Connections:
- net +3V3: now also C6.1, U5.3 (VO); no longer J1.11 (Pin_11)
- net GND: now also C5.2, C6.2, U5.4 (GND)
- new net BATT: C5.1, J1.11 (Pin_11), U5.1 (VI), U5.2 (CTL)
Other:
- moved on the sheet: C1, C2, C3, C4, J1, J2

Commit message: strain gauge hell
Other:
- company: (none) -> Manchester Stinger Motorsports
- title: (none) -> GPS and Accelerometer Carrier
Changed lines of the file:
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@@
 	(generator "eeschema")
 	(generator_version "10.0")
-	(paper "A3")
+	(paper "A4")
+	(title_block
+		(title "GPS and Accelerometer Carrier")
+		(rev "V1.0")
+		(company "Manchester Stinger Motorsports")
+		(comment 1 "James Platt")
+	)
 	(junction
 		(at 31.75 71.12)
