File: hardware/hats/Strain Gauge Interface/SGI.kicad_pcb (KiCad board)
At the start: 2 copper layers, 78 x 58 mm, 83 parts, among them IC1 ADC124S051CIMM_NOPB, IC2 ADC124S051CIMM_NOPB, J1 Conn_01x14, J2 S03B-XASK-1, J3 S03B-XASK-1, J4 S03B-XASK-1, J5 S03B-XASK-1, J6 S03B-XASK-1, J7 S03B-XASK-1, J8 S03B-XASK-1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

Commit message: update SGIH
Parts:
- added G***: LOGO, LOGO, B.Cu at (124.5, 92.1)
Other:
- board text added: "Strain Gauge Interface Hat V1.0 Designed by Agam Routed 08/05/26"

Commit message: final ordered version
Parts:
- L2: footprint customFootprints:Shielded_Inductor_SMD_7265 -> Inductor_SMD:L_Wuerth_WE-TPC-3816
- moved L2 0.82 mm to (99.8, 92.5), turned to -90 degrees
Routing:
- net +12V: track 127.9 -> 129.7 mm

Commit message: strain gauge hell
Parts:
- L2: footprint Inductor_SMD:L_Wuerth_WE-TPC-3816 -> CustomFootprints:WE-TPC_4828
- moved L2 0.49 mm to (99.3, 92.7)
