File: hardware/hats/Strain Gauge Interface V2/front/front.kicad_pcb (KiCad board)
At the start: 2 copper layers, 78 x 58 mm, 76 parts, among them J1 Conn_01x14, U1 ADS1235IRHBT, U2 ADS1235IRHBT, U3 LMR50410YQDBVRQ1, U5 BD450, U6 BD433

Commit message: this is worse than torture
Parts:
- added C38: 1nf, Capacitor_SMD:C_0603_1608Metric, F.Cu at (168.6, 146.6)
- added C39: 1nf, Capacitor_SMD:C_0603_1608Metric, F.Cu at (168.6, 149.1)
- added C40: 1nf, Capacitor_SMD:C_0603_1608Metric, F.Cu at (168.6, 151.6)
- added C41: 1nf, Capacitor_SMD:C_0603_1608Metric, F.Cu at (168.6, 154.1)
- added C42: 10nf, Capacitor_SMD:C_0603_1608Metric, F.Cu at (168.6, 156.6)
- added C43: 10nf, Capacitor_SMD:C_0603_1608Metric, F.Cu at (172.6, 146.6)
- added J2: Conn_01x07, Connector_JST:JST_XA_S07B-XASK-1_1x07_P2.50mm_Horizontal, F.Cu at (166.6, 104.6)
- added R25: 100, Resistor_SMD:R_0603_1608Metric, F.Cu at (172.6, 149.1)
- added R26: 100, Resistor_SMD:R_0603_1608Metric, F.Cu at (172.6, 151.6)
- added R27: 100, Resistor_SMD:R_0603_1608Metric, F.Cu at (172.6, 154.1)
- added R28: 100, Resistor_SMD:R_0603_1608Metric, F.Cu at (172.6, 156.6)
- added R29: 120, Resistor_SMD:R_0603_1608Metric, F.Cu at (176.7, 146.6)
- added R30: 120, Resistor_SMD:R_0603_1608Metric, F.Cu at (176.7, 149.1)
- added R31: 120, Resistor_SMD:R_0603_1608Metric, F.Cu at (176.7, 151.6)
- added R32: 120, Resistor_SMD:R_0603_1608Metric, F.Cu at (176.7, 154.1)
- added SG10: TOP, Connector_JST:JST_XA_S02B-XASK-1_1x02_P2.50mm_Horizontal, F.Cu at (116.0, 85.1)
- added SG11: BOTTOM, Connector_JST:JST_XA_S02B-XASK-1_1x02_P2.50mm_Horizontal, F.Cu at (116.0, 94.7)
- added SG12: BOTTOM, Connector_JST:JST_XA_S02B-XASK-1_1x02_P2.50mm_Horizontal, F.Cu at (118.0, 106.2)
- added SG9: TOP, Connector_JST:JST_XA_S02B-XASK-1_1x02_P2.50mm_Horizontal, F.Cu at (116.0, 75.6)
- J1: value Conn_01x14 -> Conn_01x07; footprint Connector_JST:JST_XA_S14B-XASK-1_1x14_P2.50mm_Horizontal -> Connector_JST:JST_XA_S07B-XASK-1_1x07_P2.50mm_Horizontal
- moved R2 101.8 mm to (175.6, 60.4), turned to 90 degrees
- moved C3 99.4 mm to (173.0, 62.8)
- moved C4 99.3 mm to (169.8, 63.6), turned to 180 degrees
- moved R1 96.5 mm to (175.6, 63.6), turned to 90 degrees
- moved C1 95.9 mm to (168.0, 59.0), turned to 90 degrees
- moved C6 92.6 mm to (158.4, 70.6), turned to 180 degrees
- moved C5 88.7 mm to (158.4, 72.4)
- moved C2 86.7 mm to (158.4, 67.0), turned to -90 degrees
- moved C34 83.4 mm to (158.4, 90.0)
- moved C33 79.4 mm to (158.4, 91.8), turned to 180 degrees
- moved U6 69.9 mm to (158.1, 85.5), turned to 180 degrees
- moved U5 69.6 mm to (158.0, 77.3), turned to 180 degrees
- moved J1 19.3 mm to (166.6, 83.2)
- moved U2 11.2 mm to (102.2, 143.0)
- moved U1 8.21 mm to (92.0, 139.0)
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Connections:
- J1 pad 6: unconnected-(J1-Pin_6-Pad6) -> BATT
- J1 pad 7: unconnected-(J1-Pin_7-Pad7) -> GND
- U2 pad 25: +3V3 -> AIN5_B
- U2 pad 26: +3V3 -> AIN4_B
- U2 pad 27: +3V3 -> AIN3_B
- U2 pad 28: +3V3 -> AIN2_B
Routing:
- net +6V: track 0.00 -> 53.1 mm
- net +3V3: track 0.00 -> 8.28 mm
- net Net-(U3-CB): track 0.00 -> 8.15 mm
- net Net-(U3-FB): track 0.00 -> 8.01 mm
- net BATT: track 0.00 -> 6.66 mm
- net +5V: track 0.00 -> 5.27 mm
- added copper zone on F.Cu, net Net-(U3-SW)
