File: hardware/hats/Strain Gauge Interface V2/HAT/HAT.kicad_pcb (KiCad board)
At the start: 2 copper layers, 78 x 58 mm, 95 parts, among them J1 Conn_01x07, J2 Conn_01x07, U1 ADS1235IRHBT, U2 ADS1235IRHBT, U3 LMR50410YQDBVRQ1, U5 BD450, U6 BD433

Commit message: things are looking up
Parts:
- removed C10, C17: 1uf, Capacitor_SMD:C_0603_1608Metric
- removed C16, C18, C21, C26, C29, C32, C37, C42, C43: 10nf, Capacitor_SMD:C_0603_1608Metric
- removed C19, C20, C22, C23, C24, C25, C27, C28, C30, C31, C35, C36, C38, C39, C40, C41: 1nf, Capacitor_SMD:C_0603_1608Metric
- removed R10, R11, R14, R15, R18, R19, R23, R24, R25, R26, R27, R28, R8, R9: 100, Resistor_SMD:R_0603_1608Metric
- removed R12, R13, R16, R17, R20, R21, R29, R30, R31, R32: 120, Resistor_SMD:R_0603_1608Metric
- removed R22: 100k, Resistor_SMD:R_0603_1608Metric
- removed SG1, SG10, SG3, SG5, SG7, SG9: TOP, Connector_JST:JST_XA_S02B-XASK-1_1x02_P2.50mm_Horizontal
- removed SG11, SG12, SG2, SG4, SG6, SG8: BOTTOM, Connector_JST:JST_XA_S02B-XASK-1_1x02_P2.50mm_Horizontal
- added C7: 1u, Capacitor_SMD:C_0603_1608Metric, F.Cu at (124.4, 79.6)
- added J13: BSEL, Connector_PinHeader_2.54mm:PinHeader_1x02_P2.54mm_Vertical, F.Cu at (153.6, 98.6)
- added J14: RST, Connector_PinHeader_2.54mm:PinHeader_1x02_P2.54mm_Vertical, F.Cu at (123.9, 83.2)
- added J3: Conn_01x04, Connector_JST:JST_XA_S04B-XASK-1_1x04_P2.50mm_Horizontal, F.Cu at (117.3, 83.8)
- added J4: Conn_01x04, Connector_JST:JST_XA_S04B-XASK-1_1x04_P2.50mm_Horizontal, F.Cu at (117.3, 69.8)
- added J5: Conn_01x04, Connector_JST:JST_XA_S04B-XASK-1_1x04_P2.50mm_Horizontal, F.Cu at (149.2, 67.5)
- added J6: Conn_01x04, Connector_JST:JST_XA_S04B-XASK-1_1x04_P2.50mm_Horizontal, F.Cu at (134.1, 105.3)
- added J7: Conn_01x02, Connector_JST:JST_XA_S02B-XASK-1_1x02_P2.50mm_Horizontal, F.Cu at (148.3, 105.3)
- added U4: LT1963AEST-3.3, customFootprints:SOT-223_ST_LIT, F.Cu at (158.5, 108.0)
- C11, C12: value 1uf -> 0.1u
- C13: value 1uf -> 1u
- C14, C15, C8: value 1uf -> 10u
- C9: value 10nf -> 0.1u
- J1: value Conn_01x07 -> Conn_01x14; footprint Connector_JST:JST_XA_S07B-XASK-1_1x07_P2.50mm_Horizontal -> Connector_JST:JST_XA_S14B-XASK-1_1x14_P2.50mm_Horizontal
- J2: value Conn_01x07 -> Conn_01x03; footprint Connector_JST:JST_XA_S07B-XASK-1_1x07_P2.50mm_Horizontal -> Connector_JST:JST_XA_S03B-XASK-1_1x03_P2.50mm_Horizontal
- L1: footprint CustomFootprints:WE-TPC_4828 -> customFootprints:WE-TPC_4828
- R3: value 120 -> 10k
- R4: value 100k -> 27
- R5: value 120 -> 27
- R6, R7: value 100 -> 5k1
- U1: value ADS1235IRHBT -> ESP32-S3-WROOM-1U-N4R2; footprint CustomFootprints:RHB32_TEX -> customFootprints:XCVR_ESP32-S3-WROOM-1U-N16R8
- U2: value ADS1235IRHBT -> max3392eeud+T; footprint CustomFootprints:RHB32_TEX -> customFootprints:21-0066J_14_MXM
- U3: footprint CustomFootprints:SOT95P280X145-6N -> Custom_MSM:Regulator_Switching_SOT-23-6
- moved C9 86.2 mm to (127.6, 75.1)
- moved C8 78.6 mm to (127.6, 73.4)
- moved R3 77.0 mm to (126.2, 79.6), turned to -90 degrees
- moved U1 70.5 mm to (139.3, 86.7)
- moved R7 67.1 mm to (141.6, 99.4), turned to 90 degrees
- moved R6 65.0 mm to (144.6, 99.4), turned to 90 degrees
- moved R5 59.3 mm to (135.6, 101.8), turned to -90 degrees
- moved C12 59.3 mm to (120.0, 109.4), turned to -90 degrees
- moved C11 57.1 mm to (116.4, 109.4), turned to -90 degrees
- moved R4 56.9 mm to (138.4, 101.8), turned to -90 degrees
- moved C14 55.0 mm to (165.0, 106.5)
- moved C15 54.3 mm to (165.0, 110.0)
- moved J2 49.7 mm to (117.3, 97.9), turned to -90 degrees
- moved U2 39.9 mm to (125.2, 110.4)
- moved C13 35.2 mm to (118.2, 109.4), turned to -90 degrees
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Connections:
- C11 pad 1: Net-(U1-AVDD) -> +3V3
- C12 pad 1: Net-(U1-BYPASS) -> +5V
- C13 pad 1: Net-(U2-AVDD) -> +5V
- C14 pad 1: Net-(U2-AVDD) -> +6V
- C15 pad 1: Net-(U2-BYPASS) -> +3V3EXC
- C8 pad 1: +5V -> GND
- C8 pad 2: GND -> +3V3
- C9 pad 1: Net-(U1-CAPP) -> GND
- C9 pad 2: Net-(U1-CAPN) -> +3V3
- J1 pad 1: CS1 -> 5V_CS
- J1 pad 2: CS2 -> unconnected-(J1-Pin_2-Pad2)
- J1 pad 3: SCLK -> 5V_SCLK
- J1 pad 4: DOUT -> 5V_MISO
- J1 pad 5: DIN -> 5V_MOSI
- J1 pad 6: BATT -> unconnected-(J1-Pin_6-Pad6)
- J1 pad 7: GND -> unconnected-(J1-Pin_7-Pad7)
- J2 pad 1: CS1 -> MISOSG
- J2 pad 2: CS2 -> MOSISG
- J2 pad 3: SCLK -> SCLKSG
- R3 pad 2: Net-(R3-Pad2) -> Main_Reset
- R4 pad 1: Net-(U1-REFP0) -> Net-(U1-IO19)
- R4 pad 2: Net-(U1-REFN0) -> USBD-
- R5 pad 1: GND -> Net-(U1-IO20)
- R5 pad 2: Net-(R5-Pad2) -> USBD+
- R6 pad 1: Net-(U1-REFP0) -> Net-(J6-Pin_4)
- R6 pad 2: +3V3 -> GND
- R7 pad 1: Net-(U1-REFN0) -> Net-(J6-Pin_3)
- U1 pad 1: unconnected-(U1-NC-Pad1) -> GND
- U1 pad 10: CS1 -> CSB1
- U1 pad 11: SCLK -> CSB2
- U1 pad 12: DIN -> unconnected-(U1-IO8-Pad12)
- U1 pad 13: unconnected-(U1-*DRDY-Pad13) -> Net-(U1-IO19)
- U1 pad 14: DOUT -> Net-(U1-IO20)
- U1 pad 15: Net-(U1-BYPASS) -> unconnected-(U1-IO3-Pad15)
- U1 pad 16: GND -> unconnected-(U1-IO46-Pad16)
- U1 pad 17: +5V -> unconnected-(U1-IO9-Pad17)
- U1 pad 18: GND -> CSA
- U1 pad 19: unconnected-(U1-NC-Pad19) -> MOSIA
- U1 pad 2: Net-(U1-CAPP) -> +3V3
- U1 pad 20: unconnected-(U1-NC-Pad20) -> SCLKA
- U1 pad 21: unconnected-(U1-NC-Pad21) -> MISOA
- U1 pad 22: unconnected-(U1-NC-Pad22) -> SCLKSG
- U1 pad 23: unconnected-(U1-NC-Pad23) -> CSB3
- U1 pad 25: AIN5_A -> unconnected-(U1-IO48-Pad25)
- U1 pad 26: AIN4_A -> unconnected-(U1-IO45-Pad26)
- U1 pad 27: AIN3_A -> Net-(J13-Pin_2)
- U1 pad 28: AIN2_A -> CSB4
- U1 pad 29: AIN1_A -> CSB5
- U1 pad 3: Net-(U1-CAPN) -> Main_Reset
- U1 pad 30: AIN0_A -> CSB6
- U1 pad 31: Net-(U1-REFN0) -> CSB7
- U1 pad 32: Net-(U1-REFP0) -> unconnected-(U1-IO39-Pad32)
- U1 pad 33: GND -> unconnected-(U1-IO40-Pad33)
- U1 pad 4: Net-(U1-AVDD) -> unconnected-(U1-IO4-Pad4)
- U1 pad 5: GND -> unconnected-(U1-IO5-Pad5)
- U1 pad 7: +5V -> unconnected-(U1-IO7-Pad7)
- U1 pad 8: +5V -> MOSISG
- U1 pad 9: +5V -> MISOSG
- U2 pad 1: unconnected-(U2-NC-Pad1) -> +3V3
- U2 pad 10: CS2 -> 5V_MISO
- U2 pad 11: SCLK -> 5V_SCLK
- U2 pad 12: DIN -> 5V_MOSI
- U2 pad 13: unconnected-(U2-*DRDY-Pad13) -> 5V_CS
- U2 pad 14: DOUT -> +5V
- U2 pad 2: Net-(U2-CAPP) -> CSA
- U2 pad 3: Net-(U2-CAPN) -> MOSIA
- U2 pad 4: Net-(U2-AVDD) -> SCLKA
- U2 pad 5: GND -> MISOA
- U2 pad 7: +5V -> GND
- U2 pad 8: +5V -> +3V3
- U2 pad 9: +5V -> unconnected-(U2-NC-Pad9)
Routing:
- net +3V3: track 8.28 -> 112.6 mm, vias 0 -> 3
- net +5V: track 5.27 -> 88.0 mm
- net 5V_MISO: track 0.00 -> 65.3 mm
- net 5V_MOSI: track 0.00 -> 64.1 mm, vias 0 -> 1
- net 5V_SCLK: track 0.00 -> 62.5 mm
- net +3V3EXC: track 0.00 -> 60.0 mm, vias 0 -> 1
- net CSB5: track 0.00 -> 55.4 mm
- net 5V_CS: track 0.00 -> 54.5 mm
- net CSB6: track 0.00 -> 53.8 mm
- net CSB7: track 0.00 -> 51.5 mm
- net MOSISG: track 0.00 -> 34.4 mm
- net CSB4: track 0.00 -> 31.9 mm, vias 0 -> 2
- net CSB3: track 0.00 -> 28.8 mm, vias 0 -> 2
- net SCLKSG: track 0.00 -> 28.5 mm, vias 0 -> 2
- net MISOA: track 0.00 -> 24.2 mm
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- added copper zone on B.Cu, net GND
- added copper zone on F.Cu, net GND
Other:
- board text added: "IO0"
- board text added: "MReset"

Commit message: its finally over
Parts:
- added G***: LOGO, LOGO, B.Cu at (142.2, 90.2)
- U4: footprint customFootprints:SOT-223_ST_LIT -> Package_TO_SOT_SMD:SOT-223-3_TabPin2
- moved U4 0.25 mm to (158.2, 108.0), turned to 0 degrees
Routing:
- net +6V: track 63.4 -> 85.2 mm
- net GND: vias 11 -> 17
Other:
- board text added: "Strain Gauge Hat V2"
