File: hardware/hats/Strain Gauge Interface V2/HAT/HAT.kicad_sch (KiCad schematic)
At the start: 31 parts, among them J1 Conn_01x14, J13 BSEL, J14 RST, J2 Conn_01x03, J3 Conn_01x04, J4 Conn_01x04, U1 ESP32-S3-WROOM-1U-N4R2, U2 max3392eeud+T, U3 LMR50410YQDBVRQ1, U5 BD450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

Commit message: connector
Parts:
- added J5: Conn_01x03, symbol Connector_Generic:Conn_01x03
Connections:
- net +3V3: now also J5.2 (Pin_2)
- net +5V: now also J5.1 (Pin_1)
- net GND: now also J5.3 (Pin_3)

Commit message: things are looking up
Parts:
- removed J5: Conn_01x03, symbol Connector_Generic:Conn_01x03
- added C14, C15: 10u, Capacitor_SMD:C_0603_1608Metric, symbol Device:C
- added J5, J6: Conn_01x04, Connector_JST:JST_XA_S04B-XASK-1_1x04_P2.50mm_Horizontal, symbol Connector_Generic:Conn_01x04
- added J7: Conn_01x02, Connector_JST:JST_XA_S02B-XASK-1_1x02_P2.50mm_Horizontal, symbol Connector_Generic:Conn_01x02
- added R6, R7: 5k1, Resistor_SMD:R_0603_1608Metric, symbol Device:R
- added U4: LT1963AEST-3.3, customFootprints:SOT-223_ST_LIT, symbol LT1963AEST-3.3:LT1963AEST-3.3
- J1: footprint (none) -> Connector_JST:JST_XA_S14B-XASK-1_1x14_P2.50mm_Horizontal
- J2: footprint (none) -> Connector_JST:JST_XA_S03B-XASK-1_1x03_P2.50mm_Horizontal
- J3, J4: footprint (none) -> Connector_JST:JST_XA_S04B-XASK-1_1x04_P2.50mm_Horizontal
- L1: footprint CustomFootprints:WE-TPC_4828 -> customFootprints:WE-TPC_4828
- U1: footprint CustomFootprints:XCVR_ESP32-S3-WROOM-1U-N4R2 -> customFootprints:XCVR_ESP32-S3-WROOM-1U-N16R8
- U2: footprint 21-0066J_14_MXM -> customFootprints:21-0066J_14_MXM
- U3: footprint CustomFootprints:SOT95P280X145-6N -> Custom_MSM:Regulator_Switching_SOT-23-6
Connections:
- net 5V_DIN is gone; now on net 5V_MOSI: J1.5 (Pin_5)
- net 5V_DOUT is gone; now on net 5V_MISO: J1.4 (Pin_4)
- net +3V3: now also J5.1 (Pin_1)
- net +5V: now also J5.2 (Pin_2), J7.2 (Pin_2)
- net +6V: now also C14.1, U4.1 (IN)
- net GND: now also C14.2, C15.2, J5.4 (Pin_4), J7.1 (Pin_1), R6.2, R7.2, U4.2 (GND)
- net USBD+: now also J6.1 (Pin_1)
- net USBD-: now also J6.2 (Pin_2)
- new net: J6.3 (Pin_3), R7.1
- new net: J6.4 (Pin_4), R6.1
- new net +3V3EXC: C15.1, J5.3 (Pin_3), U4.3 (OUT)

Commit message: its finally over
Parts:
- U4: footprint customFootprints:SOT-223_ST_LIT -> Package_TO_SOT_SMD:SOT-223-3_TabPin2
