File: hardware/hats/Strain Gauge Interface V2/TEENY_ROSETTE/TEENY_ROSETTE.kicad_pcb (KiCad board)
At the start: 2 copper layers, 33 x 33 mm, 61 parts, among them J1 Conn_01x01, J10 Conn_01x01, J11 Conn_01x01, J12 Conn_01x01, J13 Conn_01x01, J14 Conn_01x01, J15 Conn_01x01, J16 Conn_01x01, J17 Conn_01x01, J18 Conn_01x01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

Commit message: its finally over
Parts:
- removed J15, J16, J19, J20, J21, J22: Conn_01x01, CustomFootprints10:PAD
- added R18: 120, Resistor_SMD:R_0603_1608Metric, F.Cu at (155.1, 69.4)
- added R19: 120, Resistor_SMD:R_0603_1608Metric, F.Cu at (163.5, 71.5)
- added R20: 120, Resistor_SMD:R_0603_1608Metric, F.Cu at (175.2, 68.7)
Routing:
- net GND: track 16.1 -> 15.2 mm
- net Net-(J23-Pin_1): track 11.3 -> 12.1 mm
- net Net-(R15-Pad2): vias 1 -> 2
- net Net-(R20-Pad1): vias 1 -> 2
- net Net-(R11-Pad2): vias 1 -> 2
