File: hardware/hats/Strain Gauge Interface V2/TEENY_ROSETTE/TEENY_ROSETTE.kicad_sch (KiCad schematic)
At the start: 60 parts, among them J1 Conn_01x01, J10 Conn_01x01, J11 Conn_01x01, J12 Conn_01x01, J13 Conn_01x01, J14 Conn_01x01, J15 Conn_01x01, J16 Conn_01x01, J17 Conn_01x01, J18 Conn_01x01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

Commit message: its finally over
Parts:
- removed J15, J16, J19, J20, J21, J22: Conn_01x01, CustomFootprints10:PAD, symbol Connector_Generic:Conn_01x01
- added R18, R19, R20: 120, Resistor_SMD:R_0603_1608Metric, symbol Device:R_45deg
Connections:
- net GND: now also R18.1, R19.2, R20.2
- net at R15.2, R17.2: now also R18.2
- net at R3.2, R8.2: now also R20.1
- net at R11.2, R13.2: now also R19.1
